Commit message: Upgrade IsaacSim 5.1 / IsaacLab 2.3 (requires Python 3.11) You need to reset your Conda environment: 1. Run scripts/reset_isaacsim.sh to remove existing IsaacSim and IsaacLab installs 2. Run scripts/setup_isaacsim.sh Unitree SDK version is bumped for Python 3.11 to support sim2sim:   source scripts/source_isaacsim_setup.sh   python -m holosoma.run_sim simulator:isaacsim Updated virtual gantry to use non-deprecated quat_apply_inverse().
Source-Commit: 154c5c3

File: src/holosoma/holosoma/data/robots/g1/g1_29dof.urdf (robot description, URDF)
Before this commit: robot g1, 42 links, 41 joints
Links:
- link LL_FOOT: geometry visual box size=0.001 0.001 0.001
- link LR_FOOT: geometry visual box size=0.001 0.001 0.001
- link imu_in_pelvis: geometry visual box size=0.001 0.001 0.001
- link imu_in_torso: geometry visual box size=0.001 0.001 0.001
- link left_foot_contact_point: geometry visual box size=0.001 0.001 0.001
- link mid360_link: geometry visual box size=0.001 0.001 0.001
- link right_foot_contact_point: geometry visual box size=0.001 0.001 0.001

File: src/holosoma/holosoma/data/robots/t1/t1_29dof.urdf (robot description, URDF)
Before this commit: robot T1, 32 links, 31 joints
Links:
- link left_foot_contact_point: geometry visual box size=0.001 0.001 0.001
- link right_foot_contact_point: geometry visual box size=0.001 0.001 0.001
