Commit message: Revise isaacsim

File: src/holosoma/holosoma/data/robots/statue_v0_1/statue_v0_1.urdf (robot description, URDF)
Before this commit: robot statue_main_for_urdf_w_waist, 32 links, 31 joints
Links:
- link left_ankle_pitch_link: geometry collision mesh filename=package://statue_v0_1/meshes/left_ankle_pitch_link.STL; visual mesh filename=package://statue_v0_1/meshes/left_ankle_pitch_link.STL
- link left_ankle_roll_link: geometry collision mesh filename=package://statue_v0_1/meshes/left_ankle_roll_link.STL; visual mesh filename=package://statue_v0_1/meshes/left_ankle_roll_link.STL
- link left_elbow_pitch_link: geometry collision mesh filename=package://statue_v0_1/meshes/left_elbow_pitch_link.STL; visual mesh filename=package://statue_v0_1/meshes/left_elbow_pitch_link.STL
- link left_hip_pitch_link: geometry collision mesh filename=package://statue_v0_1/meshes/left_hip_pitch_link.STL; visual mesh filename=package://statue_v0_1/meshes/left_hip_pitch_link.STL
- link left_hip_roll_link: geometry collision mesh filename=package://statue_v0_1/meshes/left_hip_roll_link.STL; visual mesh filename=package://statue_v0_1/meshes/left_hip_roll_link.STL
- link left_hip_yaw_link: geometry collision mesh filename=package://statue_v0_1/meshes/left_hip_yaw_link.STL; visual mesh filename=package://statue_v0_1/meshes/left_hip_yaw_link.STL
- link left_knee_pitch_link: geometry collision mesh filename=package://statue_v0_1/meshes/left_knee_pitch_link.STL; visual mesh filename=package://statue_v0_1/meshes/left_knee_pitch_link.STL
- link left_shoulder_pitch_link: geometry collision mesh filename=package://statue_v0_1/meshes/left_shoulder_pitch_link.STL; visual mesh filename=package://statue_v0_1/meshes/left_shoulder_pitch_link.STL
- link left_shoulder_roll_link: geometry collision mesh filename=package://statue_v0_1/meshes/left_shoulder_roll_link.STL; visual mesh filename=package://statue_v0_1/meshes/left_shoulder_roll_link.STL
- link left_shoulder_yaw_link: geometry collision mesh filename=package://statue_v0_1/meshes/left_shoulder_yaw_link.STL; visual mesh filename=package://statue_v0_1/meshes/left_shoulder_yaw_link.STL
- link left_wrist_pitch_link: geometry collision mesh filename=package://statue_v0_1/meshes/left_welder.STL; visual mesh filename=package://statue_v0_1/meshes/left_welder.STL
- link left_wrist_roll_link: geometry collision mesh filename=package://statue_v0_1/meshes/left_wrist_roll_link.STL; visual mesh filename=package://statue_v0_1/meshes/left_wrist_roll_link.STL
- link left_wrist_yaw_link: geometry collision mesh filename=package://statue_v0_1/meshes/left_wrist_yaw_link.STL; visual mesh filename=package://statue_v0_1/meshes/left_wrist_yaw_link.STL
- link pelvis_link: geometry collision mesh filename=package://statue_v0_1/meshes/pelvis_link.STL; visual mesh filename=package://statue_v0_1/meshes/pelvis_link.STL
- link right_ankle_pitch_link: geometry collision mesh filename=package://statue_v0_1/meshes/right_ankle_pitch_link.STL; visual mesh filename=package://statue_v0_1/meshes/right_ankle_pitch_link.STL
- link right_ankle_roll_link: geometry collision mesh filename=package://statue_v0_1/meshes/right_ankle_roll_link.STL; visual mesh filename=package://statue_v0_1/meshes/right_ankle_roll_link.STL
- link right_elbow_pitch_link: geometry collision mesh filename=package://statue_v0_1/meshes/right_elbow_pitch_link.STL; visual mesh filename=package://statue_v0_1/meshes/right_elbow_pitch_link.STL
- link right_hip_pitch_link: geometry collision mesh filename=package://statue_v0_1/meshes/right_hip_pitch_link.STL; visual mesh filename=package://statue_v0_1/meshes/right_hip_pitch_link.STL
- link right_hip_roll_link: geometry collision mesh filename=package://statue_v0_1/meshes/right_hip_roll_link.STL; visual mesh filename=package://statue_v0_1/meshes/right_hip_roll_link.STL
- link right_hip_yaw_link: geometry collision mesh filename=package://statue_v0_1/meshes/right_hip_yaw_link.STL; visual mesh filename=package://statue_v0_1/meshes/right_hip_yaw_link.STL
- link right_knee_pitch_link: geometry collision mesh filename=package://statue_v0_1/meshes/right_knee_pitch_link.STL; visual mesh filename=package://statue_v0_1/meshes/right_knee_pitch_link.STL
- link right_shoulder_pitch_link: geometry collision mesh filename=package://statue_v0_1/meshes/right_shoulder_pitch_link.STL; visual mesh filename=package://statue_v0_1/meshes/right_shoulder_pitch_link.STL
- link right_shoulder_roll_link: geometry collision mesh filename=package://statue_v0_1/meshes/right_shoulder_roll_link.STL; visual mesh filename=package://statue_v0_1/meshes/right_shoulder_roll_link.STL
- link right_shoulder_yaw_link: geometry collision mesh filename=package://statue_v0_1/meshes/right_shoulder_yaw_link.STL; visual mesh filename=package://statue_v0_1/meshes/right_shoulder_yaw_link.STL
- link right_wrist_pitch_link: geometry collision mesh filename=package://statue_v0_1/meshes/right_welder.STL; visual mesh filename=package://statue_v0_1/meshes/right_welder.STL
- link right_wrist_roll_link: geometry collision mesh filename=package://statue_v0_1/meshes/right_wrist_roll_link.STL; visual mesh filename=package://statue_v0_1/meshes/right_wrist_roll_link.STL
- link right_wrist_yaw_link: geometry collision mesh filename=package://statue_v0_1/meshes/right_wrist_yaw_link.STL; visual mesh filename=package://statue_v0_1/meshes/right_wrist_yaw_link.STL
- link waist_pitch_link: geometry collision mesh filename=package://statue_v0_1/meshes/waist_pitch_link.STL; visual mesh filename=package://statue_v0_1/meshes/waist_pitch_link.STL
- link waist_roll_link: geometry collision mesh filename=package://statue_v0_1/meshes/waist_roll_link.STL; visual mesh filename=package://statue_v0_1/meshes/waist_roll_link.STL
- link waist_yaw_link: geometry collision mesh filename=package://statue_v0_1/meshes/waist_yaw_link.STL; visual mesh filename=package://statue_v0_1/meshes/waist_yaw_link.STL
