Commit message: 成功实现wbt的数据重映射

File: src/holosoma/holosoma/data/robots/h1/h1.urdf (robot description, URDF)
Before this commit: robot h1, 20 links, 19 joints
Links:
- added link d435_left_imager_link; collision sphere radius=0.001; visual sphere radius=0.001
- added link d435_rgb_module_link; collision sphere radius=0.001; visual sphere radius=0.001
- added link imu_link
- added link left_foot_contact_point, mass 0.001
- added link logo_link; visual mesh filename=package://h1_description/meshes/logo_link.STL
- added link mid360_link; collision sphere radius=0.001; visual sphere radius=0.001
- added link right_foot_contact_point, mass 0.001
- link left_ankle_link: mass 0.446 -> 0.725; geometry collision box size=0.28 0.03 0.024; visual mesh filename=package://h1_description/meshes/left_ankle_link.STL
- link left_elbow_link: mass 0.669 -> 0.745; geometry collision cylinder length=0.09 radius=0.03; visual mesh filename=package://h1_description/meshes/left_elbow_link.STL
- link left_hip_pitch_link: mass 4.152 -> 4.953; geometry collision cylinder length=0.2 radius=0.05; visual mesh filename=package://h1_description/meshes/left_hip_pitch_link.STL
- link left_hip_roll_link: mass 2.232 -> 2.7150; geometry collision cylinder length=0.01 radius=0.02; visual mesh filename=package://h1_description/meshes/left_hip_roll_link.STL
- link left_hip_yaw_link: mass 2.244 -> 2.965; geometry collision cylinder length=0.02 radius=0.01; visual mesh filename=package://h1_description/meshes/left_hip_yaw_link.STL
- link left_knee_link: mass 1.721 -> 2.824; geometry collision cylinder length=0.2 radius=0.05; visual mesh filename=package://h1_description/meshes/left_knee_link.STL
- link left_shoulder_pitch_link: mass 1.033 -> 1.142; geometry collision cylinder length=0.04 radius=0.03; visual mesh filename=package://h1_description/meshes/left_shoulder_pitch_link.STL
- link left_shoulder_roll_link: mass 0.793 -> 0.852; geometry collision cylinder length=0.01 radius=0.04; visual mesh filename=package://h1_description/meshes/left_shoulder_roll_link.STL
- link left_shoulder_yaw_link: mass 0.839 -> 0.862; geometry collision cylinder length=0.01 radius=0.04; visual mesh filename=package://h1_description/meshes/left_shoulder_yaw_link.STL
- link pelvis: mass 5.39 -> 5.983; geometry collision sphere radius=0.05; visual mesh filename=package://h1_description/meshes/pelvis.STL
- link right_ankle_link: mass 0.446 -> 0.725; geometry collision box size=0.28 0.03 0.024; visual mesh filename=package://h1_description/meshes/right_ankle_link.STL
- link right_elbow_link: mass 0.669 -> 0.745; geometry collision cylinder length=0.09 radius=0.03; visual mesh filename=package://h1_description/meshes/right_elbow_link.STL
- link right_hip_pitch_link: mass 4.152 -> 4.953; geometry collision cylinder length=0.2 radius=0.05; visual mesh filename=package://h1_description/meshes/right_hip_pitch_link.STL
- link right_hip_roll_link: mass 2.232 -> 2.7150; geometry collision cylinder length=0.01 radius=0.02; visual mesh filename=package://h1_description/meshes/right_hip_roll_link.STL
- link right_hip_yaw_link: mass 2.244 -> 2.965; geometry collision cylinder length=0.02 radius=0.01; visual mesh filename=package://h1_description/meshes/right_hip_yaw_link.STL
- link right_knee_link: mass 1.721 -> 2.824; geometry collision cylinder length=0.2 radius=0.05; visual mesh filename=package://h1_description/meshes/right_knee_link.STL
- link right_shoulder_pitch_link: mass 1.033 -> 1.142; geometry collision cylinder length=0.04 radius=0.03; visual mesh filename=package://h1_description/meshes/right_shoulder_pitch_link.S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
- link right_shoulder_roll_link: mass 0.793 -> 0.852; geometry collision cylinder length=0.01 radius=0.04; visual mesh filename=package://h1_description/meshes/right_shoulder_roll_link.STL
- link right_shoulder_yaw_link: mass 0.839 -> 0.862; geometry collision cylinder length=0.01 radius=0.04; visual mesh filename=package://h1_description/meshes/right_shoulder_yaw_link.STL
- link torso_link: geometry collision box size=0.08 0.16 0.1; visual mesh filename=package://h1_description/meshes/torso_link.STL
Joints:
- added joint d435_left_imager_joint: type fixed, parent torso_link, child d435_left_imager_link, origin xyz=0.10848474394 0.0175 0.69317107367 rpy=-2.45735 0 -1.57080, axis 0 0 0
- added joint d435_rgb_module_joint: type fixed, parent torso_link, child d435_rgb_module_link, origin xyz=0.10848474394 0.0325 0.69317107367 rpy=-2.45735 0 -1.57080, axis 0 0 0
- added joint imu_joint: type fixed, parent torso_link, child imu_link, origin xyz=-0.04452 -0.01891 0.27756 rpy=0 0 0
- added joint left_foot_contact_point_joint: type fixed, parent left_ankle_link, child left_foot_contact_point, origin xyz=0.055 0 -0.07 rpy=0 0 0
- added joint logo_joint: type fixed, parent torso_link, child logo_link, origin xyz=0 0 0 rpy=0 0 0, axis 0 0 0
- added joint mid360_joint: type fixed, parent torso_link, child mid360_link, origin xyz=0.04729990180 0 0.67492878653 rpy=0 0.243124 0, axis 0 0 0
- added joint right_foot_contact_point_joint: type fixed, parent right_ankle_link, child right_foot_contact_point, origin xyz=0.055 0 -0.07 rpy=0 0 0
- joint left_hip_pitch_joint: limit lower=-1.57 upper=1.57 effort=200 velocity=23 -> lower=-3.14 upper=2.53 effort=200 velocity=23
- joint right_hip_pitch_joint: limit lower=-1.57 upper=1.57 effort=200 velocity=23 -> lower=-3.14 upper=2.53 effort=200 velocity=23

File: src/holosoma_retargeting/holosoma_retargeting/models/h1/h1_19dof.urdf (robot description, URDF)
Before this commit: robot h1_19dof, 39 links, 38 joints
Links:
- removed link left_ankle_intermediate_link
- removed link left_foot_sphere_1_link
- removed link left_foot_sphere_2_link
- removed link left_foot_sphere_3_link
- removed link left_foot_sphere_4_link
- removed link left_foot_sphere_5_link
- removed link left_hand_sphere_link
- removed link right_ankle_intermediate_link
- removed link right_foot_sphere_1_link
- removed link right_foot_sphere_2_link
- removed link right_foot_sphere_3_link
- removed link right_foot_sphere_4_link
- removed link right_foot_sphere_5_link
- removed link right_hand_sphere_link
- added link left_foot_contact_point, mass 0.001
- added link right_foot_contact_point, mass 0.001
- link left_ankle_link: mass 0.474 -> 0.725; geometry collision box size=0.28 0.03 0.024; visual mesh filename=package://h1_description/meshes/left_ankle_link.STL
- link left_elbow_link: mass 0.723 -> 0.745; geometry collision cylinder length=0.09 radius=0.03; visual mesh filename=package://h1_description/meshes/left_elbow_link.STL
- link left_hip_pitch_link: mass 4.152 -> 4.953; geometry collision cylinder length=0.2 radius=0.05; visual mesh filename=package://h1_description/meshes/left_hip_pitch_link.STL
- link left_hip_roll_link: mass 2.232 -> 2.7150; geometry collision cylinder length=0.01 radius=0.02; visual mesh filename=package://h1_description/meshes/left_hip_roll_link.STL
- link left_hip_yaw_link: mass 2.244 -> 2.965; geometry collision cylinder length=0.02 radius=0.01; visual mesh filename=package://h1_description/meshes/left_hip_yaw_link.STL
- link left_knee_link: mass 1.721 -> 2.824; geometry collision cylinder length=0.2 radius=0.05; visual mesh filename=package://h1_description/meshes/left_knee_link.STL
- link left_shoulder_pitch_link: mass 1.033 -> 1.142; geometry collision cylinder length=0.04 radius=0.03; visual mesh filename=package://h1_description/meshes/left_shoulder_pitch_link.STL
- link left_shoulder_roll_link: mass 0.793 -> 0.852; geometry collision cylinder length=0.01 radius=0.04; visual mesh filename=package://h1_description/meshes/left_shoulder_roll_link.STL
- link left_shoulder_yaw_link: mass 0.839 -> 0.862; geometry collision cylinder length=0.01 radius=0.04; visual mesh filename=package://h1_description/meshes/left_shoulder_yaw_link.STL
- link logo_link: geometry visual mesh filename=package://h1_description/meshes/logo_link.STL
- link pelvis: mass 5.39 -> 5.983; geometry collision sphere radius=0.05; visual mesh filename=package://h1_description/meshes/pelvis.STL
- link right_ankle_link: mass 0.474 -> 0.725; geometry collision box size=0.28 0.03 0.024; visual mesh filename=package://h1_description/meshes/right_ankle_link.STL
- link right_elbow_link: mass 0.723 -> 0.745; geometry collision cylinder length=0.09 radius=0.03; visual mesh filename=package://h1_description/meshes/right_elbow_link.STL
- link right_hip_pitch_link: mass 4.152 -> 4.953; geometry collision cylinder length=0.2 radius=0.05; visual mesh filename=package://h1_description/meshes/right_hip_pitch_link.STL
- link right_hip_roll_link: mass 2.232 -> 2.7150; geometry collision cylinder length=0.01 radius=0.02; visual mesh filename=package://h1_description/meshes/right_hip_roll_link.STL
- link right_hip_yaw_link: mass 2.244 -> 2.965; geometry collision cylinder length=0.02 radius=0.01; visual mesh filename=package://h1_description/meshes/right_hip_yaw_link.STL
- link right_knee_link: mass 1.721 -> 2.824; geometry collision cylinder length=0.2 radius=0.05; visual mesh filename=package://h1_description/meshes/right_knee_link.STL
- link right_shoulder_pitch_link: mass 1.033 -> 1.142; geometry collision cylinder length=0.04 radius=0.03; visual mesh filename=package://h1_description/meshes/right_shoulder_pitch_link.S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
- link right_shoulder_roll_link: mass 0.793 -> 0.852; geometry collision cylinder length=0.01 radius=0.04; visual mesh filename=package://h1_description/meshes/right_shoulder_roll_link.STL
- link right_shoulder_yaw_link: mass 0.839 -> 0.862; geometry collision cylinder length=0.01 radius=0.04; visual mesh filename=package://h1_description/meshes/right_shoulder_yaw_link.STL
- link torso_link: geometry collision box size=0.08 0.16 0.1; visual mesh filename=package://h1_description/meshes/torso_link.STL
Joints:
- removed joint left_ankle_intermediate_joint
- removed joint left_foot_sphere_1_joint
- removed joint left_foot_sphere_2_joint
- removed joint left_foot_sphere_3_joint
- removed joint left_foot_sphere_4_joint
- removed joint left_foot_sphere_5_joint
- removed joint left_hand_sphere_joint
- removed joint right_ankle_intermediate_joint
- removed joint right_foot_sphere_1_joint
- removed joint right_foot_sphere_2_joint
- removed joint right_foot_sphere_3_joint
- removed joint right_foot_sphere_4_joint
- removed joint right_foot_sphere_5_joint
- removed joint right_hand_sphere_joint
- added joint left_foot_contact_point_joint: type fixed, parent left_ankle_link, child left_foot_contact_point, origin xyz=0.055 0 -0.07 rpy=0 0 0
- added joint right_foot_contact_point_joint: type fixed, parent right_ankle_link, child right_foot_contact_point, origin xyz=0.055 0 -0.07 rpy=0 0 0
